Commit message: jackal with laser etc

File: jackal_description/urdf/accessories.urdf.xacro (robot description, xacro)
@@ -106,33 +106,3 @@
     </joint>
   </xacro:if>
-  <xacro:include filename="$(find jackal_description)/urdf/accessories/hokuyo_ust10.urdf.xacro" />
-  <xacro:if value="$(optenv JACKAL_FRONT_ACCESSORY_FENDER 0)">
-    <xacro:if value="$(optenv JACKAL_FRONT_FENDER_UST10 0)">
-        <hokuyo_ust10 prefix="front_ust10" parent_link="front_fender_accessory_link"/>
-    </xacro:if>
-  </xacro:if>
-  <xacro:if value="$(optenv JACKAL_REAR_ACCESSORY_FENDER 0)">
-    <xacro:if value="$(optenv JACKAL_REAR_FENDER_UST10 0)">
-        <hokuyo_ust10 prefix="rear_ust10" parent_link="rear_fender_accessory_link"/>
-    </xacro:if>
-  </xacro:if>
-  <xacro:if value="$(optenv JACKAL_ARK_ENCLOSURE 0)">
-    <link name="ark_enclosure_link">
-      <visual>
-        <origin xyz="0 0 0" rpy="0 0 0"/>
-        <geometry>
-          <mesh filename="package://jackal_description/meshes/ark_enclosure.stl"/>
-        </geometry>
-        <material name="dark_grey" />
-      </visual>
-    </link>
-    <joint name="ark_enclosure_joint" type="fixed">
-      <parent link="mid_mount" />
-      <child link="ark_enclosure_link" />
-    </joint>
-    <gazebo reference="ark_enclosure_link">
-      <material>Gazebo/DarkGrey</material>
-      <turnGravityOff>false</turnGravityOff>
-    </gazebo>
-  </xacro:if>
 </robot>

File: jackal_description/urdf/accessories/bridge_plate.urdf.xacro (robot description, xacro)
@@ -1,4 +1,4 @@
 <?xml version="1.0"?>
-<robot xmlns:xacro="http://www.ros.org/wiki/xacro">
+<robot xmlns:xacro="http://ros.org/wiki/xacro">
   <xacro:macro name="bridge_plate" params="mount height">
     <joint name="${mount}_mount_to_${mount}_bridge" type="fixed">

File: jackal_description/urdf/accessories/camera_mount.urdf.xacro (robot description, xacro)
@@ -1,3 +1,3 @@
-<robot xmlns:xacro="http://www.ros.org/wiki/xacro">
+<robot xmlns:xacro="http://ros.org/wiki/xacro">
   <xacro:macro name="camera_mount" params="prefix tilt:=0">
     <link name="${prefix}_camera_mount">

File: jackal_description/urdf/accessories/novatel_smart6.urdf.xacro (robot description, xacro)
@@ -1,4 +1,4 @@
 <?xml version="1.0"?>
-<robot xmlns:xacro="http://www.ros.org/wiki/xacro">
+<robot xmlns:xacro="http://ros.org/wiki/xacro">
   <xacro:macro name="novatel_smart6" params="prefix">
   <link name="${prefix}_navsat">

File: jackal_description/urdf/accessories/sick_lms1xx_mount.urdf.xacro (robot description, xacro)
@@ -25,5 +25,5 @@
 SOFTWARE, EVEN IF ADVISED OF THE POSSIBILITY OF SUCH DAMAGE.
 -->
-<robot xmlns:xacro="http://www.ros.org/wiki/xacro">
+<robot xmlns:xacro="http://ros.org/wiki/xacro">
   <xacro:include filename="$(find lms1xx)/urdf/sick_lms1xx.urdf.xacro" />
   <xacro:macro name="sick_lms1xx_mount" params="prefix topic">

File: jackal_description/urdf/accessories/stereo_camera_mount.urdf.xacro (robot description, xacro)
@@ -1,3 +1,3 @@
-<robot xmlns:xacro="http://www.ros.org/wiki/xacro">
+<robot xmlns:xacro="http://ros.org/wiki/xacro">
   <xacro:macro name="stereo_camera_mount" params="prefix tilt:=0">
     <link name="${prefix}_stereo_camera_mount" />

File: jackal_description/urdf/jackal2.urdf.xacro (robot description, xacro)
@@ -12,10 +12,15 @@
   <xacro:property name="chassis_height" value="0.184" />
   <xacro:property name="dummy_inertia" value="1e-09"/>
-  <xacro:property name="mount_spacing" value="0.120" />
+  <xacro:property name="mount_spacing" value="0.115" />
+  <xacro:property name="velodyne_height" value="0.5" />
+  <xacro:property name="long_beam" value="0.35" />
+  <xacro:property name="short_beam" value="0.135" />
+  <xacro:property name="plate_thickness" value="0.005" />
   <material name="dark_grey"><color rgba="0.2 0.2 0.2 1.0" /></material>
   <material name="light_grey"><color rgba="0.4 0.4 0.4 1.0" /></material>
   <material name="yellow"><color rgba="0.8 0.8 0.0 1.0" /></material>
   <material name="black"><color rgba="0.15 0.15 0.15 1.0" /></material>
-  <xacro:macro name="wheel" params="prefix *joint_pose">
+  <material name="alu"><color rgba="0.56 0.56 0.56 1.0" /></material>
+<xacro:macro name="wheel" params="prefix *joint_pose">
     <link name="${prefix}_wheel_link">
       <visual>
@@ -55,8 +60,8 @@
       <type>transmission_interface/SimpleTransmission</type>
       <joint name="${prefix}_wheel">
-        <hardwareInterface>VelocityJointInterface</hardwareInterface>
+        <hardwareInterface>hardware_interface/VelocityJointInterface</hardwareInterface>
       </joint>
       <actuator name="${prefix}_actuator">
-        <mechanicalReduction>1</mechanicalReduction>
+        <mechanicalReduction>10</mechanicalReduction>
       </actuator>
     </transmission>
@@ -160,16 +165,195 @@
     <origin xyz="${-mount_spacing} 0 0" />
   </joint>
+  <joint name="front_mount_joint" type="fixed">
+    <parent link="mid_mount" />
+    <child link="hokuyo_base_link" />
+    <origin xyz="${mount_spacing} 0 0.015" />
+  </joint>
   <link name="front_mount"></link>
-  <joint name="front_mount_joint" type="fixed">
+  <joint name="front_mount_joint_2" type="fixed">
     <parent link="mid_mount" />
     <child link="front_mount" />
     <origin xyz="${mount_spacing} 0 0" />
   </joint>
+  <joint name="baseplate_mount_joint" type="fixed">
+    <parent link="mid_mount"/>
+    <child link="baseplate_link"/>
+    <origin xyz="0 0 0.01"/>
+  </joint>
+  <link name="baseplate_link">
+    <visual>
+      <origin xyz="0.05 0 ${plate_thickness/2}" rpy="0 0 0"/>
+      <geometry>
+        <box size="0.3 0.3 ${plate_thickness}" />
+      </geometry>
+      <material name="alu" />
+    </visual>
+    <visual>
+      <origin xyz="-0.15 0 ${plate_thickness/2}" rpy="0 0 0"/>
+      <geometry>
+        <box size="0.1 0.16 ${plate_thickness}"/>
+      </geometry>
+      <material name="alu"/>
+    </visual>
+    <visual>
+      <origin xyz="-0.077 -0.105 ${long_beam/2 + plate_thickness}" rpy="0 0 0"/>
+      <geometry>
+        <box size="0.03 0.03 ${long_beam}" />
+      </geometry>
+      <material name="alu" />
+    </visual>
+    <visual>
+      <origin xyz="0.038 -0.105 ${long_beam/2 + plate_thickness}" rpy="0 0 0"/>
+      <geometry>
+        <box size="0.03 0.03 ${long_beam}" />
+      </geometry>
+      <material name="alu" />
+    </visual>
+    <visual>
+      <origin xyz="-0.077 0.105 ${long_beam/2 + plate_thickness}" rpy="0 0 0"/>
+      <geometry>
+        <box size="0.03 0.03 ${long_beam}" />
+      </geometry>
+      <material name="alu" />
+    </visual>
+    <visual>
+      <origin xyz="0.038 0.105 ${long_beam/2 + plate_thickness}" rpy="0 0 0"/>
+      <geometry>
+        <box size="0.03 0.03 ${long_beam}" />
+      </geometry>
+      <material name="alu" />
+    </visual>
+    <visual>
+      <origin xyz="-0.0195 0 ${long_beam + 3*plate_thickness/2}" rpy="0 0 0"/>
+      <geometry>
+        <box size="0.145 0.24 ${plate_thickness}" />
+      </geometry>
+      <material name="alu" />
+    </visual>
+<!-- SHORT BEAMS -->
+    <visual>
+      <origin xyz="-0.077 -0.07 ${long_beam + short_beam/2 + 2*plate_thickness}" rpy="0 0 0"/>
+      <geometry>
+        <box size="0.03 0.03 ${short_beam}" />
+      </geometry>
+      <material name="alu" />
+    </visual>
+    <visual>
+      <origin xyz="0.038 -0.07 ${long_beam + short_beam/2 + 2*plate_thickness}" rpy="0 0 0"/>
+      <geometry>
+        <box size="0.03 0.03 ${short_beam}" />
+      </geometry>
+      <material name="alu" />
+    </visual>
+    <visual>
+      <origin xyz="-0.077 0.07 ${long_beam + short_beam/2 + 2*plate_thickness}" rpy="0 0 0"/>
+      <geometry>
+        <box size="0.03 0.03 ${short_beam}" />
+      </geometry>
+      <material name="alu" />
+    </visual>
+    <visual>
+      <origin xyz="0.038 0.07 ${long_beam + short_beam/2 + 2*plate_thickness}" rpy="0 0 0"/>
+      <geometry>
+        <box size="0.03 0.03 ${short_beam}" />
+      </geometry>
+      <material name="alu" />
+    </visual>
+    <visual>
+      <origin xyz="-0.0195 0 ${long_beam + short_beam + 5*plate_thickness/2}" rpy="0 0 0"/>
+      <geometry>
+        <box size="0.145 0.17 ${plate_thickness}" />
+      </geometry>
+      <material name="alu" />
+    </visual>
+  </link>
+  <link name="hokuyo_base_link">
+    <visual>
+      <origin xyz="0 0 0.0205" rpy="0 0 0"/>
+      <geometry>
+        <box size="0.05 0.05 0.041"/>
+      </geometry>
+      <material name="black"/>
+    </visual>
+    <visual>
+      <origin xyz="-0.021 0 0.049" rpy="0 0 0"/>
+      <geometry>
+        <box size="0.008 0.012 0.022"/>
+      </geometry>
+      <material name="black"/>
+    </visual>
+    <visual>
+      <origin xyz="0 0 0.06" rpy="0 0 0"/>
+      <geometry>
+        <cylinder radius="0.019" length="0.02"/>
+      </geometry>
+      <material name="black"/>
+    </visual>
+    <visual>
+      <origin xyz="0 0 0.0455" rpy="0 0 0"/>
+      <geometry>
+        <cylinder radius="0.021" length="0.009"/>
+      </geometry>
+      <material name="black"/>
+    </visual>
+  </link>
+  <link name="hokuyo_base_scan"></link>
+  <joint name="hokuyo_base_scan_joint" type="fixed" >
+       <origin xyz="0 0 0.0563" rpy="0 0 0" />
+       <parent link="hokuyo_base_link" />
+       <child link="hokuyo_base_scan"/>
+  </joint>
+  <joint name="$VLP16_base_mount_joint" type="fixed">
+      <parent link="mid_mount"/>
+      <child link="VLP16_base_link"/>
+      <origin xyz="0 0 ${velodyne_height + 0.01}" />
+  </joint>
+  <link name="VLP16_base_link">
+      <inertial>
+        <mass value="0.1"/>
+       <origin xyz="0 0 0"/>
+        <inertia ixx="0.1" ixy="0" ixz="0" iyy="0.1" iyz="0" izz="0.1"/>
+      </inertial>
+      <visual>
+        <geometry>
+          <mesh filename="package://velodyne_description/meshes/VLP16_base_1.dae" />
+        </geometry>
+      </visual>
+      <visual>
+        <geometry>
+          <mesh filename="package://velodyne_description/meshes/VLP16_base_2.dae" />
+        </geometry>
+      </visual>
+      <collision>
+        <origin rpy="0 0 0" xyz="0 0 0.03585"/>
+        <geometry>
+          <cylinder radius="0.0516" length="0.0717"/>
+        </geometry>
+      </collision>
+  </link>
+  <joint name="VLP16_base_scan_joint" type="fixed" >
+       <origin xyz="0 0 0.0377" rpy="0 0 0" />
+       <parent link="VLP16_base_link" />
+       <child link="VLP16"/>
+  </joint>
+  <link name="VLP16">
+      <inertial>
+        <mass value="0.1"/>
+        <origin xyz="0 0 0"/>
+        <inertia ixx="0.1" ixy="0" ixz="0" iyy="0.1" iyz="0" izz="0.1"/>
+      </inertial>
+      <visual>
+        <origin xyz="0 0 -0.0377" />
+        <geometry>
+          <mesh filename="package://velodyne_description/meshes/VLP16_scan.dae" />
+        </geometry>
+      </visual>
+  </link>
   <!-- Bring in simulation data for Gazebo. -->
-  <xacro:include filename="$(find jackal_description)/urdf/jackal.gazebo" />
+  <xacro:include filename="jackal.gazebo" />
   <!-- Optional standard accessories, including their simulation data. The rendering
        of these into the final description is controlled by optenv variables, which
        default each one to off.-->
-  <xacro:include filename="$(find jackal_description)/urdf/accessories.urdf.xacro" />
+  <xacro:include filename="accessories.urdf.xacro" />
   <!-- Optional custom includes. -->
   <xacro:include filename="$(optenv JACKAL_URDF_EXTRAS empty.urdf)" />

File: jackal_description/urdf/jackal_sensor.urdf.xacro (robot description, xacro)
@@ -12,10 +12,15 @@
   <xacro:property name="chassis_height" value="0.184" />
   <xacro:property name="dummy_inertia" value="1e-09"/>
-  <xacro:property name="mount_spacing" value="0.120" />
+  <xacro:property name="mount_spacing" value="0.115" />
+  <xacro:property name="velodyne_height" value="0.5" />
+  <xacro:property name="long_beam" value="0.35" />
+  <xacro:property name="short_beam" value="0.135" />
+  <xacro:property name="plate_thickness" value="0.005" />
   <material name="dark_grey"><color rgba="0.2 0.2 0.2 1.0" /></material>
   <material name="light_grey"><color rgba="0.4 0.4 0.4 1.0" /></material>
   <material name="yellow"><color rgba="0.8 0.8 0.0 1.0" /></material>
   <material name="black"><color rgba="0.15 0.15 0.15 1.0" /></material>
-  <xacro:macro name="wheel" params="prefix *joint_pose">
+  <material name="alu"><color rgba="0.56 0.56 0.56 1.0" /></material>
+<xacro:macro name="wheel" params="prefix *joint_pose">
     <link name="${prefix}_wheel_link">
       <visual>
@@ -160,16 +165,189 @@
     <origin xyz="${-mount_spacing} 0 0" />
   </joint>
-  <link name="front_mount"></link>
   <joint name="front_mount_joint" type="fixed">
     <parent link="mid_mount" />
-    <child link="front_mount" />
-    <origin xyz="${mount_spacing} 0 0" />
-  </joint>
+    <child link="hokuyo_base_link" />
+    <origin xyz="${mount_spacing} 0 0.015" />
+  </joint>
+  <joint name="baseplate_mount_joint" type="fixed">
+    <parent link="mid_mount"/>
+    <child link="baseplate_link"/>
+    <origin xyz="0 0 0.01"/>
+  </joint>
+  <link name="baseplate_link">
+    <visual>
+      <origin xyz="0.05 0 ${plate_thickness/2}" rpy="0 0 0"/>
+      <geometry>
+        <box size="0.3 0.3 ${plate_thickness}" />
+      </geometry>
+      <material name="alu" />
+    </visual>
+    <visual>
+      <origin xyz="-0.15 0 ${plate_thickness/2}" rpy="0 0 0"/>
+      <geometry>
+        <box size="0.1 0.16 ${plate_thickness}"/>
+      </geometry>
+      <material name="alu"/>
+    </visual>
+    <visual>
+      <origin xyz="-0.077 -0.105 ${long_beam/2 + plate_thickness}" rpy="0 0 0"/>
+      <geometry>
+        <box size="0.03 0.03 ${long_beam}" />
+      </geometry>
+      <material name="alu" />
+    </visual>
+    <visual>
+      <origin xyz="0.038 -0.105 ${long_beam/2 + plate_thickness}" rpy="0 0 0"/>
+      <geometry>
+        <box size="0.03 0.03 ${long_beam}" />
+      </geometry>
+      <material name="alu" />
+    </visual>
+    <visual>
+      <origin xyz="-0.077 0.105 ${long_beam/2 + plate_thickness}" rpy="0 0 0"/>
+      <geometry>
+        <box size="0.03 0.03 ${long_beam}" />
+      </geometry>
+      <material name="alu" />
+    </visual>
+    <visual>
+      <origin xyz="0.038 0.105 ${long_beam/2 + plate_thickness}" rpy="0 0 0"/>
+      <geometry>
+        <box size="0.03 0.03 ${long_beam}" />
+      </geometry>
+      <material name="alu" />
+    </visual>
+    <visual>
+      <origin xyz="-0.0195 0 ${long_beam + 3*plate_thickness/2}" rpy="0 0 0"/>
+      <geometry>
+        <box size="0.145 0.24 ${plate_thickness}" />
+      </geometry>
+      <material name="alu" />
+    </visual>
+<!-- SHORT BEAMS -->
+    <visual>
+      <origin xyz="-0.077 -0.07 ${long_beam + short_beam/2 + 2*plate_thickness}" rpy="0 0 0"/>
+      <geometry>
+        <box size="0.03 0.03 ${short_beam}" />
+      </geometry>
+      <material name="alu" />
+    </visual>
+    <visual>
+      <origin xyz="0.038 -0.07 ${long_beam + short_beam/2 + 2*plate_thickness}" rpy="0 0 0"/>
+      <geometry>
+        <box size="0.03 0.03 ${short_beam}" />
+      </geometry>
+      <material name="alu" />
+    </visual>
+    <visual>
+      <origin xyz="-0.077 0.07 ${long_beam + short_beam/2 + 2*plate_thickness}" rpy="0 0 0"/>
+      <geometry>
+        <box size="0.03 0.03 ${short_beam}" />
+      </geometry>
+      <material name="alu" />
+    </visual>
+    <visual>
+      <origin xyz="0.038 0.07 ${long_beam + short_beam/2 + 2*plate_thickness}" rpy="0 0 0"/>
+      <geometry>
+        <box size="0.03 0.03 ${short_beam}" />
+      </geometry>
+      <material name="alu" />
+    </visual>
+    <visual>
+      <origin xyz="-0.0195 0 ${long_beam + short_beam + 5*plate_thickness/2}" rpy="0 0 0"/>
+      <geometry>
+        <box size="0.145 0.17 ${plate_thickness}" />
+      </geometry>
+      <material name="alu" />
+    </visual>
+  </link>
+  <link name="hokuyo_base_link">
+    <visual>
+      <origin xyz="0 0 0.0205" rpy="0 0 0"/>
+      <geometry>
+        <box size="0.05 0.05 0.041"/>
+      </geometry>
+      <material name="black"/>
+    </visual>
+    <visual>
+      <origin xyz="-0.021 0 0.049" rpy="0 0 0"/>
+      <geometry>
+        <box size="0.008 0.012 0.022"/>
+      </geometry>
+      <material name="black"/>
+    </visual>
+    <visual>
+      <origin xyz="0 0 0.06" rpy="0 0 0"/>
+      <geometry>
+        <cylinder radius="0.019" length="0.02"/>
+      </geometry>
+      <material name="black"/>
+    </visual>
+    <visual>
+      <origin xyz="0 0 0.0455" rpy="0 0 0"/>
+      <geometry>
+        <cylinder radius="0.021" length="0.009"/>
+      </geometry>
+      <material name="black"/>
+    </visual>
+  </link>
+  <link name="hokuyo_base_scan"></link>
+  <joint name="hokuyo_base_scan_joint" type="fixed" >
+       <origin xyz="0 0 0.0563" rpy="0 0 0" />
+       <parent link="hokuyo_base_link" />
+       <child link="hokuyo_base_scan"/>
+  </joint>
+  <joint name="$VLP16_base_mount_joint" type="fixed">
+      <parent link="mid_mount"/>
+      <child link="VLP16_base_link"/>
+      <origin xyz="0 0 ${velodyne_height + 0.01}" />
+  </joint>
+  <link name="VLP16_base_link">
+      <inertial>
+        <mass value="0.1"/>
+       <origin xyz="0 0 0"/>
+        <inertia ixx="0.1" ixy="0" ixz="0" iyy="0.1" iyz="0" izz="0.1"/>
+      </inertial>
+      <visual>
+        <geometry>
+          <mesh filename="package://velodyne_description/meshes/VLP16_base_1.dae" />
+        </geometry>
+      </visual>
+      <visual>
+        <geometry>
+          <mesh filename="package://velodyne_description/meshes/VLP16_base_2.dae" />
+        </geometry>
+      </visual>
+      <collision>
+        <origin rpy="0 0 0" xyz="0 0 0.03585"/>
+        <geometry>
+          <cylinder radius="0.0516" length="0.0717"/>
+        </geometry>
+      </collision>
+  </link>
+  <joint name="VLP16_base_scan_joint" type="fixed" >
+       <origin xyz="0 0 0.0377" rpy="0 0 0" />
+       <parent link="VLP16_base_link" />
+       <child link="VLP16"/>
+  </joint>
+  <link name="VLP16">
+      <inertial>
+        <mass value="0.1"/>
+        <origin xyz="0 0 0"/>
+        <inertia ixx="0.1" ixy="0" ixz="0" iyy="0.1" iyz="0" izz="0.1"/>
+      </inertial>
+      <visual>
+        <origin xyz="0 0 -0.0377" />
+        <geometry>
+          <mesh filename="package://velodyne_description/meshes/VLP16_scan.dae" />
+        </geometry>
+      </visual>
+  </link>
   <!-- Bring in simulation data for Gazebo. -->
-  <xacro:include filename="$(find jackal_description)/urdf/jackal.gazebo" />
+  <xacro:include filename="jackal.gazebo" />
   <!-- Optional standard accessories, including their simulation data. The rendering
        of these into the final description is controlled by optenv variables, which
        default each one to off.-->
-  <xacro:include filename="$(find jackal_description)/urdf/accessories.urdf.xacro" />
+  <xacro:include filename="accessories.urdf.xacro" />
   <!-- Optional custom includes. -->
   <xacro:include filename="$(optenv JACKAL_URDF_EXTRAS empty.urdf)" />
